File: kicad/diff-line-demo/diff-line-demo.kicad_pcb (KiCad board)
At the start: 4 copper layers, 177.7 x 343 mm, 2 parts, among them J1 HDMI_A, J2 HDMI_A

Commit message: Revert "Pricing of larger board."
This reverts commit 5b3cc41474cecd1aedfbfebfedbf0e034cb78ffa.
Other:
- board size 177.7 x 343 mm -> 177.7 x 137.7 mm
Changed lines of the file:
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@@
 	(gr_rect
 		(start 50.8508 40)
-		(end 228.6 383.0066)
+		(end 228.6 177.673)
 		(stroke
 			(width 0.05)
@@
 		(polygon
 			(pts
-				(xy 50.8 40) (xy 228.6 40) (xy 228.6 383.3622) (xy 50.8 383.3622)
+				(xy 50.8 40) (xy 228.6 40) (xy 228.6 177.673) (xy 50.8 177.673)
 			)
 		)

Commit message: Pricing of larger board.
Other:
- board size 177.7 x 137.7 mm -> 177.7 x 343 mm
Changed lines of the file:
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@@
 	(gr_rect
 		(start 50.8508 40)
-		(end 228.6 177.673)
+		(end 228.6 383.0066)
 		(stroke
 			(width 0.05)
@@
 		(polygon
 			(pts
-				(xy 50.8 40) (xy 228.6 40) (xy 228.6 177.673) (xy 50.8 177.673)
+				(xy 50.8 40) (xy 228.6 40) (xy 228.6 383.3622) (xy 50.8 383.3622)
 			)
 		)
